File: kicad_files/gas67_plus.kicad_sch (KiCad schematic)
At the start: 33 parts, among them J1 USB_C_Receptacle_USB2.0, SW1 SW_Push, U1 W25Q128JVS, U2 AP2112K-3.3, U3 RP2040, Y1 12MHz

Commit message: Added LED and switch matrices.
Parts:
- added C18, C19, C20, C21, C22, C23, C24, C25, C26, C27, C28, C29, C30, C31, C32, C33, C34, C35, C36, C37, C38, C39, C40, C41, C42, C43, C44, C45, C46, C47, C48, C49, C50, C51, C52, C53, C54, C55, C56, C57, C58, C59, C60, C61, C62, C63, C64, C65, C66, C67, C68, C69, C70, C71, C72, C73, C74, C75, C76, C77, C78, C79, C80, C81, C82, C83, C84, C85, C86, C87, C88, C89, C90, C91, C92: 100nF, symbol Device:C_Small
- added D10, D11, D12, D13, D14, D15, D16, D17, D18, D19, D2, D20, D21, D22, D23, D24, D25, D26, D27, D28, D29, D3, D30, D31, D32, D33, D34, D35, D36, D37, D38, D39, D4, D40, D41, D42, D43, D44, D45, D46, D47, D48, D49, D5, D50, D51, D52, D53, D54, D55, D56, D57, D58, D59, D6, D60, D61, D62, D63, D64, D67, D68, D69, D7, D71, D72, D73, D74, D75, D76, D8, D9: D_Small, symbol Device:D_Small
- added D100, D101, D102, D103, D104, D105, D106, D107, D108, D109, D110, D111, D112, D113, D114, D115, D116, D117, D118, D119, D120, D121, D122, D123, D124, D125, D126, D127, D128, D129, D130, D131, D132, D133, D134, D135, D136, D137, D138, D139, D140, D141, D142, D143, D144, D145, D146, D147, D148, D65, D66, D70, D77, D78, D79, D80, D81, D82, D83, D84, D85, D86, D87, D88, D89, D90, D91, D92, D93, D94, D95, D96, D97, D98, D99: SK6812MINI, LED_SMD:LED_SK6812MINI_PLCC4_3.5x3.5mm_P1.75mm, symbol LED:SK6812MINI
- added MX1, MX10, MX11, MX12, MX13, MX14, MX15, MX16, MX17, MX18, MX19, MX2, MX20, MX21, MX22, MX23, MX24, MX25, MX26, MX27, MX28, MX29, MX3, MX30, MX31, MX32, MX33, MX34, MX35, MX36, MX37, MX38, MX39, MX4, MX40, MX41, MX42, MX43, MX44, MX45, MX46, MX47, MX48, MX49, MX5, MX50, MX51, MX52, MX53, MX54, MX55, MX56, MX57, MX58, MX59, MX6, MX60, MX61, MX62, MX63, MX64, MX65, MX66, MX67, MX68, MX69, MX7, MX70, MX71, MX72, MX73, MX74, MX75, MX76, MX77, MX8, MX9: MX_SW_HS, PCM_marbastlib-mx:SW_MX_HS_1u, symbol marbastlib-mx:MX_SW_HS
- added Q1: BSS138, Package_TO_SOT_SMD:SOT-23, symbol Transistor_FET:BSS138
- added R10, R11, R12, R13, R14, R15, R16, R17, R18, R19, R20, R21, R22, R23, R24, R25, R26, R27, R28, R29, R30, R31, R32, R33, R34, R35, R36, R37, R38, R39, R40, R41, R42, R43, R44, R45, R46, R47, R48, R49, R50, R51, R52, R53, R54, R55, R56, R57, R58, R59, R60, R61, R62, R63, R64, R65, R66, R67, R68, R69, R70, R71, R72, R73, R74, R75, R76, R77, R78, R79, R80, R81, R82, R83, R84: 5.1R, symbol Device:R_Small_US
- added R8, R9: 10k, symbol Device:R_Small_US
Connections:
- net +3V3: now also Q1.1 (G), R8.2
- net +5V: now also R10.2, R11.2, R12.2, R13.2, R14.2, R15.2, R16.2, R17.2, R18.2, R19.2, R20.2, R21.2, R22.2, R23.2, R24.2, R25.2, R26.2, R27.2, R28.2, R29.2, R30.2, R31.2, R32.2, R33.2, R34.2, R35.2, R36.2, R37.2, R38.2, R39.2, R40.2, R41.2, R42.2, R43.2, R44.2, R45.2, R46.2, R47.2, R48.2, R49.2, R50.2, R51.2, R52.2, R53.2, R54.2, R55.2, R56.2, R57.2, R58.2, R59.2, R60.2, R61.2, R62.2, R63.2, R64.2, R65.2, R66.2, R67.2, R68.2, R69.2, R70.2, R71.2, R72.2, R73.2, R74.2, R75.2, R76.2, R77.2, R78.2, R79.2, R80.2, R81.2, R82.2, R83.2, R84.2, R9.2
- net GND: now also C18.2, C19.2, C20.2, C21.2, C22.2, C23.2, C24.2, C25.2, C26.2, C27.2, C28.2, C29.2, C30.2, C31.2, C32.2, C33.2, C34.2, C35.2, C36.2, C37.2, C38.2, C39.2, C40.2, C41.2, C42.2, C43.2, C44.2, C45.2, C46.2, C47.2, C48.2, C49.2, C50.2, C51.2, C52.2, C53.2, C54.2, C55.2, C56.2, C57.2, C58.2, C59.2, C60.2, C61.2, C62.2, C63.2, C64.2, C65.2, C66.2, C67.2, C68.2, C69.2, C70.2, C71.2, C72.2, C73.2, C74.2, C75.2, C76.2, C77.2, C78.2, C79.2, C80.2, C81.2, C82.2, C83.2, C84.2, C85.2, C86.2, C87.2, C88.2, C89.2, C90.2, C91.2, C92.2, D100.2 (VSS), D101.2 (VSS), D102.2 (VSS), D103.2 (VSS), D104.2 (VSS), D105.2 (VSS), D106.2 (VSS), D107.2 (VSS), D108.2 (VSS), D109.2 (VSS), D110.2 (VSS), D111.2 (VSS), D112.2 (VSS), D113.2 (VSS), D114.2 (VSS), D115.2 (VSS), D116.2 (VSS), D117.2 (VSS), D118.2 (VSS), D119.2 (VSS), D120.2 (VSS), D121.2 (VSS), D122.2 (VSS), D123.2 (VSS), D124.2 (VSS), D125.2 (VSS), D126.2 (VSS), D127.2 (VSS), D128.2 (VSS), D129.2 (VSS), D130.2 (VSS), D131.2 (VSS), D132.2 (VSS), D133.2 (VSS), D134.2 (VSS), D135.2 (VSS), D136.2 (VSS), D137.2 (VSS), D138.2 (VSS), D139.2 (VSS), D140.2 (VSS), D141.2 (VSS), D142.2 (VSS), D143.2 (VSS), D144.2 (VSS), D145.2 (VSS), D146.2 (VSS), D147.2 (VSS), D148.2 (VSS), D65.2 (VSS), D66.2 (VSS), D70.2 (VSS), D77.2 (VSS), D78.2 (VSS), D79.2 (VSS), D80.2 (VSS), D81.2 (VSS), D82.2 (VSS), D83.2 (VSS), D84.2 (VSS), D85.2 (VSS), D86.2 (VSS), D87.2 (VSS), D88.2 (VSS), D89.2 (VSS), D90.2 (VSS), D91.2 (VSS), D92.2 (VSS), D93.2 (VSS), D94.2 (VSS), D95.2 (VSS), D96.2 (VSS), D97.2 (VSS), D98.2 (VSS), D99.2 (VSS)
- new net: D73.2 (A), MX72.2
- new net: D147.1 (DOUT), D148.3 (DIN)
- new net: D146.1 (DOUT), D147.3 (DIN)
- new net: C91.1, D147.4 (VDD), R83.1
- new net: D33.2 (A), MX32.2
- new net: C22.1, D78.4 (VDD), R14.1
- new net: C40.1, D96.4 (VDD), R32.1
- new net: C50.1, D106.4 (VDD), R42.1
- new net: D36.2 (A), MX35.2
- new net: D103.1 (DOUT), D104.3 (DIN)
- new net: D103.3 (DIN), D99.1 (DOUT)
- new net: C47.1, D103.4 (VDD), R39.1
- new net: C32.1, D88.4 (VDD), R24.1
- new net: C92.1, D148.4 (VDD), R84.1
- new net: C82.1, D138.4 (VDD), R74.1
- new net: D137.1 (DOUT), D138.3 (DIN)
- new net: D136.1 (DOUT), D137.3 (DIN)
- new net: C81.1, D137.4 (VDD), R73.1
- new net: D87.1 (DOUT), D88.3 (DIN)
- new net: D86.1 (DOUT), D87.3 (DIN)
- new net: C31.1, D87.4 (VDD), R23.1
- new net: D41.2 (A), MX40.2
- new net: D50.2 (A), MX49.2
- new net: D90.1 (DOUT), D92.3 (DIN)
- new net: D89.1 (DOUT), D90.3 (DIN)
- new net: C34.1, D90.4 (VDD), R26.1
- new net: C35.1, D91.4 (VDD), R27.1
- new net: D138.1 (DOUT), D139.3 (DIN)
- new net: C74.1, D130.4 (VDD), R66.1
- new net: D38.2 (A), MX37.2
- new net: D4.2 (A), MX3.2
- new net: C85.1, D141.4 (VDD), R77.1
- new net: D23.2 (A), MX22.2
- new net: C78.1, D134.4 (VDD), R70.1
- new net: C39.1, D95.4 (VDD), R31.1
- new net: D51.2 (A), MX50.2
- new net: C29.1, D85.4 (VDD), R21.1
- new net: D75.2 (A), MX74.2
- new net: C90.1, D146.4 (VDD), R82.1
- new net: C84.1, D140.4 (VDD), R76.1
- new net: C71.1, D127.4 (VDD), R63.1
- new net: C19.1, D66.4 (VDD), R11.1
- new net: D58.2 (A), MX57.2
- new net: D104.1 (DOUT), D105.3 (DIN)
- new net: C48.1, D104.4 (VDD), R40.1
- new net: D119.1 (DOUT), D134.3 (DIN)
- new net: D119.3 (DIN), D120.1 (DOUT)
- new net: C63.1, D119.4 (VDD), R55.1
- new net: C23.1, D79.4 (VDD), R15.1
- new net: D105.1 (DOUT), D106.3 (DIN)
- new net: C49.1, D105.4 (VDD), R41.1
- new net: C72.1, D128.4 (VDD), R64.1
- new net: D17.2 (A), MX16.2
- new net: D93.1 (DOUT), D98.3 (DIN)
- new net: D93.3 (DIN), D94.1 (DOUT)
- new net: C37.1, D93.4 (VDD), R29.1
- new net: C28.1, D84.4 (VDD), R20.1
- new net: D144.1 (DOUT), D145.3 (DIN)
- new net: D143.1 (DOUT), D144.3 (DIN)
- new net: C88.1, D144.4 (VDD), R80.1
- new net: D44.2 (A), MX43.2
- new net: D91.1 (DOUT), D94.3 (DIN)
- new net: C38.1, D94.4 (VDD), R30.1
- new net: D126.3 (DIN), D127.1 (DOUT)
- new net: D127.3 (DIN), D128.1 (DOUT)
- new net: C36.1, D92.4 (VDD), R28.1
- new net: D100.3 (DIN), D101.1 (DOUT)
- new net: D101.3 (DIN), D102.1 (DOUT)
- new net: C45.1, D101.4 (VDD), R37.1
- new net: C64.1, D120.4 (VDD), R56.1
- new net: D67.2 (A), MX66.2
- new net: D27.2 (A), MX26.2
- new net: C30.1, D86.4 (VDD), R22.1
- new net: D32.2 (A), MX31.2, MX76.2
- new net: D54.2 (A), MX53.2
- new net: C26.1, D82.4 (VDD), R18.1
- new net: D97.3 (DIN), D98.1 (DOUT)
- new net: C42.1, D98.4 (VDD), R34.1
- new net: D26.2 (A), MX25.2
- new net: D76.2 (A), MX75.2
- new net: D128.3 (DIN), D129.1 (DOUT)
- new net: D129.3 (DIN), D130.1 (DOUT)
- new net: C73.1, D129.4 (VDD), R65.1
- new net: C79.1, D135.4 (VDD), R71.1
- new net: D43.2 (A), MX42.2
- new net: C41.1, D97.4 (VDD), R33.1
- new net: D35.2 (A), MX34.2
- new net: D48.2 (A), MX47.2
- new net: D111.1 (DOUT), D112.3 (DIN)
- new net: D110.1 (DOUT), D111.3 (DIN)
- new net: C55.1, D111.4 (VDD), R47.1
- new net: D6.2 (A), MX5.2
- new net: D2.2 (A), MX1.2
- new net: C57.1, D113.4 (VDD), R49.1
- new net: D19.2 (A), MX18.2
- new net: C43.1, D99.4 (VDD), R35.1
- new net: D55.2 (A), MX54.2
- new net: C76.1, D132.4 (VDD), R68.1
- new net: D102.3 (DIN), D95.1 (DOUT)
- new net: D95.3 (DIN), D96.1 (DOUT)
- new net: C80.1, D136.4 (VDD), R72.1
- new net: C56.1, D112.4 (VDD), R48.1
- new net: C61.1, D117.4 (VDD), R53.1
- new net: C68.1, D124.4 (VDD), R60.1
- new net: C62.1, D118.4 (VDD), R54.1
- new net: D85.1 (DOUT), D86.3 (DIN)
- new net: D11.2 (A), MX10.2
- new net: C59.1, D115.4 (VDD), R51.1
- new net: D34.2 (A), MX33.2
- new net: C46.1, D102.4 (VDD), R38.1
- new net: D8.2 (A), MX7.2
- new net: D30.2 (A), MX29.2
- new net: D91.3 (DIN), D92.1 (DOUT)
- new net: D52.2 (A), MX51.2
- new net: C24.1, D80.4 (VDD), R16.1
- new net: C27.1, D83.4 (VDD), R19.1
- new net: D59.2 (A), MX58.2
- new net: D63.2 (A), MX62.2
- new net: D142.1 (DOUT), D143.3 (DIN)
- new net: D141.1 (DOUT), D142.3 (DIN)
- new net: C86.1, D142.4 (VDD), R78.1
- new net: D40.2 (A), MX39.2
- new net: D9.2 (A), MX8.2
- new net: D140.1 (DOUT), D141.3 (DIN)
- new net: D139.1 (DOUT), D140.3 (DIN)
- new net: D118.1 (DOUT), D133.3 (DIN)
- new net: D117.1 (DOUT), D118.3 (DIN)
- new net: D64.2 (A), MX63.2
- new net: C25.1, D81.4 (VDD), R17.1
- new net: C33.1, D89.4 (VDD), R25.1
- new net: C54.1, D110.4 (VDD), R46.1
- new net: D14.2 (A), MX13.2
- new net: D112.1 (DOUT), D113.3 (DIN)
- new net: D135.1 (DOUT), D136.3 (DIN)
- new net: D16.2 (A), MX15.2
- new net: C60.1, D116.4 (VDD), R52.1
- new net: D45.2 (A), MX44.2, MX69.2
- new net: D10.2 (A), MX9.2
- new net: D72.2 (A), MX71.2
- new net: C83.1, D139.4 (VDD), R75.1
- new net: C51.1, D107.4 (VDD), R43.1
- new net: D37.2 (A), MX36.2
- new net: D15.2 (A), MX14.2, MX65.2
- new net: D116.1 (DOUT), D117.3 (DIN)
- new net: D56.2 (A), MX55.2
- new net: D124.3 (DIN), D125.1 (DOUT)
- new net: D125.3 (DIN), D126.1 (DOUT)
- new net: C69.1, D125.4 (VDD), R61.1
- new net: D70.1 (DOUT), D77.3 (DIN)
- new net: D66.1 (DOUT), D70.3 (DIN)
- new net: C20.1, D70.4 (VDD), R12.1
- new net: D68.2 (A), MX64.2, MX67.2
- new net: D49.2 (A), MX48.2
- new net: C89.1, D145.4 (VDD), R81.1
- new net: D106.1 (DOUT), D107.3 (DIN)
- new net: C18.1, D65.4 (VDD), R10.1
- new net: D21.2 (A), MX20.2
- new net: D145.1 (DOUT), D146.3 (DIN)
- new net: D22.2 (A), MX21.2
- new net: D57.2 (A), MX56.2
- new net: D61.2 (A), MX60.2
- new net: C66.1, D122.4 (VDD), R58.1
- new net: D53.2 (A), MX52.2
- new net: C75.1, D131.4 (VDD), R67.1
- new net: D65.1 (DOUT), D66.3 (DIN)
- new net: D24.2 (A), MX23.2
- new net: D122.3 (DIN), D123.1 (DOUT)
- new net: D123.3 (DIN), D124.1 (DOUT)
- new net: C67.1, D123.4 (VDD), R59.1
- new net: D88.1 (DOUT), D89.3 (DIN)
- new net: D60.2 (A), MX59.2
- new net: D96.3 (DIN), D97.1 (DOUT)
- new net: C44.1, D100.4 (VDD), R36.1
- new net: D39.2 (A), MX38.2
- new net: D121.3 (DIN), D122.1 (DOUT)
- new net: C52.1, D108.4 (VDD), R44.1
- new net: D47.2 (A), MX46.2, MX77.2
- new net: C70.1, D126.4 (VDD), R62.1
- new net: D20.2 (A), MX19.2
- new net: D3.2 (A), MX2.2
- new net: D84.1 (DOUT), D85.3 (DIN)
- new net: D83.1 (DOUT), D84.3 (DIN)
- new net: D100.1 (DOUT), D99.3 (DIN)
- new net: D114.1 (DOUT), D115.3 (DIN)
- new net: D113.1 (DOUT), D114.3 (DIN)
- new net: C58.1, D114.4 (VDD), R50.1
- new net: D130.3 (DIN), D131.1 (DOUT)
- new net: D115.1 (DOUT), D116.3 (DIN)
- new net: D134.1 (DOUT), D135.3 (DIN)
- new net: D82.1 (DOUT), D83.3 (DIN)
- new net: C65.1, D121.4 (VDD), R57.1
- new net: C77.1, D133.4 (VDD), R69.1
- new net: D5.2 (A), MX4.2
- new net: D74.2 (A), MX73.2
- new net: C21.1, D77.4 (VDD), R13.1
- new net: D18.2 (A), MX17.2
- new net: D31.2 (A), MX30.2
- new net: C87.1, D143.4 (VDD), R79.1
- new net: D28.2 (A), MX27.2
- new net: D79.1 (DOUT), D80.3 (DIN)
- new net: D78.1 (DOUT), D79.3 (DIN)
- new net: D109.1 (DOUT), D110.3 (DIN)
- new net: D108.1 (DOUT), D109.3 (DIN)
- new net: C53.1, D109.4 (VDD), R45.1
- new net: D120.3 (DIN), D121.1 (DOUT)
- new net: D107.1 (DOUT), D108.3 (DIN)
- new net: D132.3 (DIN), D133.1 (DOUT)
- new net: D69.2 (A), MX68.2
- new net: D81.1 (DOUT), D82.3 (DIN)
- new net: D7.2 (A), MX6.2
- new net: D42.2 (A), MX41.2
- new net: D71.2 (A), MX70.2
- new net: D131.3 (DIN), D132.1 (DOUT)
- new net: D13.2 (A), MX12.2
- new net: D12.2 (A), MX11.2
- new net: D77.1 (DOUT), D78.3 (DIN)
- new net: D25.2 (A), MX24.2
- new net: D62.2 (A), MX61.2
- new net: D80.1 (DOUT), D81.3 (DIN)
- new net: D46.2 (A), MX45.2
- new net: D29.2 (A), MX28.2
- new net COL0: MX1.1, MX16.1, MX31.1, MX46.1, MX61.1, MX76.1, MX77.1
- new net COL1: MX17.1, MX2.1, MX32.1, MX47.1, MX62.1
- new net COL10: MX11.1, MX26.1, MX41.1, MX56.1, MX71.1
- new net COL11: MX12.1, MX27.1, MX42.1, MX57.1, MX72.1
- new net COL12: MX13.1, MX28.1, MX43.1, MX58.1, MX73.1
- new net COL13: MX14.1, MX29.1, MX44.1, MX59.1, MX65.1, MX69.1, MX74.1
- new net COL14: MX15.1, MX30.1, MX45.1, MX60.1, MX75.1
- new net COL2: MX18.1, MX3.1, MX33.1, MX48.1, MX63.1
- new net COL3: MX19.1, MX34.1, MX4.1, MX49.1
- new net COL4: MX20.1, MX35.1, MX5.1, MX50.1
- new net COL5: MX21.1, MX36.1, MX51.1, MX6.1, MX66.1
- new net COL6: MX22.1, MX37.1, MX52.1, MX64.1, MX67.1, MX7.1
- new net COL7: MX23.1, MX38.1, MX53.1, MX68.1, MX8.1
- new net COL8: MX24.1, MX39.1, MX54.1, MX9.1
- new net COL9: MX10.1, MX25.1, MX40.1, MX55.1, MX70.1
- new net RGB_3V3: Q1.2 (S), R8.1
- new net RGB_5V: D65.3 (DIN), Q1.3 (D), R9.1
- new net ROW0: D10.1 (K), D11.1 (K), D12.1 (K), D13.1 (K), D14.1 (K), D15.1 (K), D16.1 (K), D2.1 (K), D3.1 (K), D4.1 (K), D5.1 (K), D6.1 (K), D7.1 (K), D8.1 (K), D9.1 (K)
- new net ROW1: D17.1 (K), D18.1 (K), D19.1 (K), D20.1 (K), D21.1 (K), D22.1 (K), D23.1 (K), D24.1 (K), D25.1 (K), D26.1 (K), D27.1 (K), D28.1 (K), D29.1 (K), D30.1 (K), D31.1 (K)
- new net ROW2: D32.1 (K), D33.1 (K), D34.1 (K), D35.1 (K), D36.1 (K), D37.1 (K), D38.1 (K), D39.1 (K), D40.1 (K), D41.1 (K), D42.1 (K), D43.1 (K), D44.1 (K), D45.1 (K), D46.1 (K)
- new net ROW3: D47.1 (K), D48.1 (K), D49.1 (K), D50.1 (K), D51.1 (K), D52.1 (K), D53.1 (K), D54.1 (K), D55.1 (K), D56.1 (K), D57.1 (K), D58.1 (K), D59.1 (K), D60.1 (K), D61.1 (K)
- new net ROW4: D62.1 (K), D63.1 (K), D64.1 (K), D67.1 (K), D68.1 (K), D69.1 (K), D71.1 (K), D72.1 (K), D73.1 (K), D74.1 (K), D75.1 (K), D76.1 (K)
- no-connect marks 2 -> 3
Other:
- note added: "Level Shifter"
- note added: "Per-Key RGB Matrix"
- note added: "Switch Matrix"
- note added: "USB-C (pending)"
- note removed: "USB-C"
- moved on the sheet: C1, C10, C11, C12, C13, C14, C15, C16, C17, C2, C3, C4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

Commit message: Added labels to switch matrix.
Parts:
- removed Q1: BSS138, Package_TO_SOT_SMD:SOT-23, symbol Transistor_FET:BSS138
- removed R8, R9: 10k, symbol Device:R_Small_US
- added C93, C94: 100nF, symbol Device:C_Small
- added R85: 10k, symbol Device:R_Small_US
- added U4: TXS0101DBV, Package_TO_SOT_SMD:SOT-23-6, symbol Logic_LevelTranslator:TXS0101DBV
- MX1: value MX_SW_HS -> Esc
- MX10: value MX_SW_HS -> 9
- MX11: value MX_SW_HS -> 0
- MX12: value MX_SW_HS -> MINUS
- MX13: value MX_SW_HS -> EQUAL
- MX14: value MX_SW_HS -> BSPC
- MX15, MX65: value MX_SW_HS -> S_BSPC
- MX16: value MX_SW_HS -> Tab
- MX17: value MX_SW_HS -> Q
- MX18: value MX_SW_HS -> W
- MX19: value MX_SW_HS -> E
- MX2: value MX_SW_HS -> 1
- MX20: value MX_SW_HS -> R
- MX21: value MX_SW_HS -> T
- MX22: value MX_SW_HS -> Y
- MX23: value MX_SW_HS -> U
- MX24, MX38: value MX_SW_HS -> I
- MX25: value MX_SW_HS -> O
- MX26: value MX_SW_HS -> P
- MX27: value MX_SW_HS -> LBRKT
- MX28: value MX_SW_HS -> RBRKT
- MX29: value MX_SW_HS -> BSLS
- MX3: value MX_SW_HS -> 2
- MX30: value MX_SW_HS -> M1
- MX31: value MX_SW_HS -> CAPS
- MX32: value MX_SW_HS -> A
- MX33: value MX_SW_HS -> S
- MX34: value MX_SW_HS -> D
- MX35: value MX_SW_HS -> F
- MX36: value MX_SW_HS -> G
- MX37: value MX_SW_HS -> H
- MX39: value MX_SW_HS -> J
- MX4: value MX_SW_HS -> 3
- MX40: value MX_SW_HS -> K
- MX41: value MX_SW_HS -> L
- MX42: value MX_SW_HS -> COLON
- MX43: value MX_SW_HS -> QUOTE
- MX44: value MX_SW_HS -> ENTER_ANSI
- MX45: value MX_SW_HS -> M2
- MX46: value MX_SW_HS -> LSFT_ISO
- MX47: value MX_SW_HS -> GT
- MX48: value MX_SW_HS -> Z
- MX49: value MX_SW_HS -> X
- MX5: value MX_SW_HS -> 4
- MX50: value MX_SW_HS -> C
- MX51: value MX_SW_HS -> V
- MX52: value MX_SW_HS -> B
- MX53: value MX_SW_HS -> N
- MX54: value MX_SW_HS -> M
- MX55: value MX_SW_HS -> COMMA
- MX56: value MX_SW_HS -> DOT
- MX57: value MX_SW_HS -> SLSH
- MX58: value MX_SW_HS -> RSFT
- MX59: value MX_SW_HS -> UP
- MX6: value MX_SW_HS -> 5
- MX60: value MX_SW_HS -> M3
- MX61: value MX_SW_HS -> LCTRL
- MX62: value MX_SW_HS -> LGUI
- MX63: value MX_SW_HS -> LALT
- MX64, MX66, MX67, MX68: value MX_SW_HS -> SPACE
- MX69: value MX_SW_HS -> ENTER_ISO
- MX7: value MX_SW_HS -> 6
- MX70: value MX_SW_HS -> L1
- MX71: value MX_SW_HS -> L2
- MX72: value MX_SW_HS -> LEFT
- MX73: value MX_SW_HS -> DOWN
- MX74: value MX_SW_HS -> RIGHT
- MX75: value MX_SW_HS -> M4
- MX76: value MX_SW_HS -> S_CAPS
- MX77: value MX_SW_HS -> LSFT_ANSI
- MX8: value MX_SW_HS -> 7
- MX9: value MX_SW_HS -> 8
Connections:
- net +3V3: now also C93.1, R85.2, U4.1 (V_{CCA})
- net +5V: now also C94.2, U4.6 (V_{CCB})
- net GND: now also C93.2, C94.1, U4.2 (GND)
- net RGB_3V3: now also U4.3 (A)
- net RGB_5V: now also U4.4 (B)
- new net: R85.1, U4.5 (OE)
Other:
- moved on the sheet: D10, D11, D12, D13, D14, D15, D16, D17, D18, D19, D2, D20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
